Commit message: Add files via upload

File: humanoid_arm_5dof/urdf/humanoid_arm_5dof.urdf (robot description, URDF)
Before this commit: robot humanoid_arm_5dof, 34 links, 33 joints
Links:
- link 1220_m4x16_left_shoulder_yaw_screws: mass 0.00141036418698182 -> 0.0014103641869818
- link left_elbow: mass 0.779765455665873 -> 0.779765455664584
- link left_elbow_rs03_actuator: mass 0.356550890896861 -> 0.35655089089686
- link left_elbow_rs03_flange: mass 0.00407555097398881 -> 0.00407555097398886
- link left_elbow_shaft: mass 15.7008025632262 -> 16.3859228521728
- link left_hand: mass 0.285530356868975 -> 0.285530151595695
- link left_hand_rs02_flange: mass 0.00245793392108139 -> 0.0024579339210813
- link left_shoulder_pitch: mass 1.1977209978155 -> 1.19772099854413
- link left_shoulder_pitch_rs04_flange: mass 0.0075835212224452 -> 0.00758352122244511
- link left_shoulder_roll: mass 0.997620685191693 -> 0.997620680698827
- link left_shoulder_roll_rs04_actuator: mass 0.517423577893356 -> 0.517423577893354
- link left_shoulder_roll_rs04_flange: mass 0.00758352122244519 -> 0.00758352122244501
- link left_shoulder_yaw: mass 0.488068654986632 -> 0.48806958571119
- link left_shoulder_yaw_flange: mass 0.0353531461099524 -> 0.0353531461099523
- link left_shoulder_yaw_rs03_flange: mass 0.00407555097398891 -> 0.00407555097398915
- link left_shoulder_yaw_shaft: mass 0.000903649674373974 -> 0.000903649674373999
- link left_wrist: mass 0.388950905166578 -> 0.388950905166564
- link left_wrist_rs02_flange: mass 0.00245793392108131 -> 0.00245793392108132
- link left_wrist_shaft: mass 0.000903649674374008 -> 0.000903649674373992
- link m3x16_left_hand_screws: mass 0.00139374174732639 -> 0.00139374174732657
- link m3x20_left_wrist_screws: mass 0.0016213702863793 -> 0.00162137028637948
- link m4x16_eft_elbow_screws: mass 0.0027018435864776 -> 0.00270184358647751
- link m4x16_left_shoulder_yaw_screws: mass 0.0027018447469342 -> 0.00270184474693417
- link m4x20_left_wrist_screws: mass 0.00232797016313314 -> 0.00232797016313311
- link m4x25_left_elbow_screws: mass 0.002708580334445 -> 0.00270858033444492
- link m4x25_left_shoulder_screws_roll: mass 0.00451430348886326 -> 0.00451430348886333
- link m4x25_left_shoulder_yaw_screws: mass 0.00270858202481974 -> 0.0027085820248196
- link m5x22_screws_left_shoulder_pitch: mass 0.00474644340626596 -> 0.00474644340626598
- link m5x22_screws_left_shoulder_roll: mass 0.00610257053905779 -> 0.00610257053905776
Joints:
- removed joint left_elbow_rs03_flange_joint
- removed joint left_hand_rs02_flange_joint
- removed joint left_shoulder_pitch_rs04_flange_joint
- removed joint left_shoulder_roll_rs04_actuator_fixture_link
- removed joint left_shoulder_yaw_rs03_flange_joint
- removed joint left_wrist_rs02_flange_joint
- added joint left_elbow_rs03_joint: type revolute, parent left_elbow_rs03_actuator, child left_elbow_rs03_flange, origin xyz=0 0 0 rpy=0 0 0, axis 0.44287 0.89659 0, limit lower=-1.3 upper=1.9 effort=60 velocity=1.6
- added joint left_hand_rs02_joint: type revolute, parent left_hand_rs02, child left_hand_rs02_flange, origin xyz=0 0 0 rpy=0 0 0, axis 1 0 0, limit lower=-1.5 upper=1.7 effort=17 velocity=0.8
- added joint left_shoulder_pitch_rs04_joint: type revolute, parent left_shoulder_pitch_rs04_actuator, child left_shoulder_pitch_rs04_flange, origin xyz=0 0 0 rpy=0 0 0, axis 1 0 0, limit lower=-3.14 upper=3.14 effort=120 velocity=3
- added joint left_shoulder_roll_rs04_actuator_joint: type revolute, parent left_shoulder_roll_rs04_flange, child left_shoulder_roll_rs04_actuator, origin xyz=0 0 0 rpy=0 0 0, axis 0 -1 0, limit lower=-3.5 upper=0.6 effort=120 velocity=3
- added joint left_shoulder_yaw_rs03_joint: type revolute, parent left_shoulder_yaw_rs03_actuator, child left_shoulder_yaw_rs03_flange, origin xyz=0 0 0 rpy=0 0 0, axis 0 0 1, limit lower=-3.14 upper=3.14 effort=60 velocity=1.6
- added joint left_wrist_rs02_joint: type revolute, parent left_wrist_actuator, child left_wrist_rs02_flange, origin xyz=0 0 0 rpy=0 0 0, axis 0 1 0, limit lower=-3.14 upper=3.14 effort=17 velocity=0.8
- joint left_shoulder_pitch_rs04_actuator_fixture_link: origin xyz=0 0 0 rpy=0 0 0 -> xyz=0.32924 0.19509 1.45 rpy=-0.6108 0 0.53491
- joint left_shoulder_roll_rs04_flange_joint: origin xyz=0 0 0 rpy=0 0 0 -> xyz=0.11678 0.0487 -2.7056E-05 rpy=0 0 3.1416
- joint m3x20_left_wrist_screws_fixture_joint: origin xyz=0.037069 -0.024445 -0.15849 rpy=-1.2996 0 -2.0296 -> xyz=0.0370688771049235 -0.0244446769789257 -0.15848929336033 rpy=-1.29963611177836 0 -2.02959481544726
- joint m5x22_screws_left_shoulder_roll_fixture_joint: origin xyz=0.080327 0.094212 -0.026075 rpy=0.56445 0 -2.6155 -> xyz=0 0 0 rpy=0 0 0

Commit message: Add files via upload

File: humanoid_arm_5dof/urdf/humanoid_arm_5dof.urdf (robot description, URDF)
Before this commit: robot humanoid_arm_5dof, 34 links, 33 joints
Links:
- link base_fixture_link: mass 400 -> 10.0408046496141
- link left_elbow: mass 0.779765455664584 -> 0.779765455632657
- link left_elbow_rs03_flange: mass 0.00407555097398886 -> 0.00407555097398885
- link left_hand: mass 0.285530151595695 -> 0.285530357048999
- link left_hand_rs02_flange: mass 0.0024579339210813 -> 0.00245793392108137
- link left_shoulder_pitch: mass 1.19772099854413 -> 1.19772100018969
- link left_shoulder_pitch_rs04_actuator: mass 0.517423577893353 -> 0.517423577893352
- link left_shoulder_pitch_rs04_flange: mass 0.00758352122244511 -> 0.00758352122244539
- link left_shoulder_roll: mass 0.997620680698827 -> 0.997620690019998
- link left_shoulder_roll_rs04_actuator: mass 0.517423577893354 -> 0.517423577893356
- link left_shoulder_roll_rs04_flange: mass 0.00758352122244501 -> 0.00758352122244542
- link left_shoulder_yaw: mass 0.48806958571119 -> 0.488068654985182
- link left_shoulder_yaw_flange: mass 0.0353531461099523 -> 0.035353146109952
- link left_shoulder_yaw_rs03_actuator: mass 0.356550969588107 -> 0.356550969588108
- link left_shoulder_yaw_rs03_flange: mass 0.00407555097398915 -> 0.00407555097398881
- link left_shoulder_yaw_shaft: mass 0.000903649674373999 -> 0.000903649674374
- link left_wrist: mass 0.388950905166564 -> 0.38895090516656
- link left_wrist_rs02_flange: mass 0.00245793392108132 -> 0.00245793392108136
- link left_wrist_shaft: mass 0.000903649674373992 -> 0.000903649674374024
- link m3x16_left_hand_screws: mass 0.00139374174732657 -> 0.0013937417473266
- link m3x20_left_wrist_screws: mass 0.00162137028637948 -> 0.00162137028637936
- link m4x16_eft_elbow_screws: mass 0.00270184358647751 -> 0.00270184358647752
- link m4x16_left_shoulder_yaw_screws: mass 0.00270184474693417 -> 0.00270184474693413
- link m4x20_left_wrist_screws: mass 0.00232797016313311 -> 0.00232797016313296
- link m4x25_left_elbow_screws: mass 0.00270858033444492 -> 0.00270858033444496
- link m4x25_left_shoulder_screws_roll: mass 0.00451430348886333 -> 0.00451430348886338
- link m4x25_left_shoulder_yaw_screws: mass 0.0027085820248196 -> 0.00270858202481966
- link m5x22_screws_left_shoulder_pitch: mass 0.00474644340626598 -> 0.00474644340626602
- link m5x22_screws_left_shoulder_roll: mass 0.00610257053905776 -> 0.00610257053905786
Joints:
- removed joint left_shoulder_roll_rs04_actuator_joint
- added joint left_shoulder_roll_rs04_joint: type revolute, parent left_shoulder_roll_rs04_flange, child left_shoulder_roll_rs04_actuator, origin xyz=0 0 0 rpy=0 0 0, axis 0 -1 0, limit lower=-3.5 upper=0.6 effort=120 velocity=3
- joint left_elbow_rs03_joint: axis 0.44287 0.89659 0 -> 0.442871169532447 0.896585259301625 0
- joint left_hand_rs02_joint: axis 1 0 0 -> 0.999999999999999 0 0
- joint left_shoulder_pitch_rs04_actuator_fixture_link: origin xyz=0.32924 0.19509 1.45 rpy=-0.6108 0 0.53491 -> xyz=0.329242881244431 0.195085661056411 1.45000000000145 rpy=-0.61079662163343 0 0.534907346303552
- joint left_shoulder_roll_rs04_flange_joint: origin xyz=0.11678 0.0487 -2.7056E-05 rpy=0 0 3.1416 -> xyz=0.116775431275821 0.0487000000004332 -2.70558071411298E-05 rpy=0 0 3.14159265358979
- joint m3x16_left_hand_screws_fixture_joint: origin xyz=0 0.0945 0 rpy=0.64485 0.44406 0 -> xyz=0 0.0944999999998815 0 rpy=0.644848119833412 0.444064009162365 0
- joint m4x16_eft_elbow_screws_fixture_joint: origin xyz=0 0 -0.0987 rpy=0 0 2.0296 -> xyz=0 0 -0.0987000004167595 rpy=0 0 2.02959481544726

Commit message: Add files via upload

File: humanoid_arm_5dof/urdf/humanoid_arm_5dof.urdf (robot description, URDF)
Before this commit: robot humanoid_arm_5dof, 34 links, 33 joints
Links:
- link 1220_m4x16_left_shoulder_yaw_screws: mass 0.0014103641869818 -> 0.00141036418698186
- link base_fixture_link: mass 10.0408046496141 -> 400
- link left_elbow: mass 0.779765455632657 -> 0.779765455773645
- link left_elbow_rs03_actuator: mass 0.35655089089686 -> 0.356550890896857
- link left_elbow_rs03_flange: mass 0.00407555097398885 -> 0.0040755509739889
- link left_hand: mass 0.285530357048999 -> 0.285530357235036
- link left_hand_rs02_flange: mass 0.00245793392108137 -> 0.00245793392108132
- link left_shoulder_pitch: mass 1.19772100018969 -> 1.19772100042922
- link left_shoulder_pitch_rs04_flange: mass 0.00758352122244539 -> 0.00758352122244509
- link left_shoulder_roll: mass 0.997620690019998 -> 0.997620687521854
- link left_shoulder_roll_rs04_actuator: mass 0.517423577893356 -> 0.517423577893355
- link left_shoulder_roll_rs04_flange: mass 0.00758352122244542 -> 0.0075835212224449
- link left_shoulder_yaw: mass 0.488068654985182 -> 0.488068654986572
- link left_shoulder_yaw_flange: mass 0.035353146109952 -> 0.0353531461099525
- link left_shoulder_yaw_rs03_actuator: mass 0.356550969588108 -> 0.3565509695881
- link left_shoulder_yaw_rs03_flange: mass 0.00407555097398881 -> 0.00407555097398895
- link left_shoulder_yaw_shaft: mass 0.000903649674374 -> 0.000903649674373941
- link left_wrist: mass 0.38895090516656 -> 0.388950905166554
- link left_wrist_actuator: mass 0.180583065420556 -> 0.180583065420557
- link left_wrist_rs02_flange: mass 0.00245793392108136 -> 0.0024579339210813
- link left_wrist_shaft: mass 0.000903649674374024 -> 0.000903649674373958
- link m3x16_left_hand_screws: mass 0.0013937417473266 -> 0.00139374174732655
- link m3x20_left_wrist_screws: mass 0.00162137028637936 -> 0.00162137028637934
- link m4x16_eft_elbow_screws: mass 0.00270184358647752 -> 0.00270184358647755
- link m4x16_left_shoulder_yaw_screws: mass 0.00270184474693413 -> 0.00270184474693415
- link m4x20_left_wrist_screws: mass 0.00232797016313296 -> 0.00232797016313307
- link m4x25_left_elbow_screws: mass 0.00270858033444496 -> 0.00270858033444499
- link m4x25_left_shoulder_screws_roll: mass 0.00451430348886338 -> 0.00451430348886335
- link m4x25_left_shoulder_yaw_screws: mass 0.00270858202481966 -> 0.00270858202481968
- link m5x22_screws_left_shoulder_pitch: mass 0.00474644340626602 -> 0.00474644340626607
- link m5x22_screws_left_shoulder_roll: mass 0.00610257053905786 -> 0.00610257053905752
Joints:
- joint left_elbow_rs03_joint: axis 0.442871169532447 0.896585259301625 0 -> 0.442871169532446 0.896585259301625 0
- joint left_shoulder_pitch_rs04_actuator_fixture_link: origin xyz=0.329242881244431 0.195085661056411 1.45000000000145 rpy=-0.61079662163343 0 0.534907346303552 -> xyz=0.3827 -0.091826 1.4471 rpy=-0.54743 0 0
- joint m4x16_left_shoulder_yaw_screws_fixture_joint: origin xyz=-0.021972 0.0377 -0.17358 rpy=0.057123 0.11257 0.47088 -> xyz=-0.0219716026665047 0.037700000000231 -0.173578614834026 rpy=0.0571232457871902 0.112571265320765 0.47087557604578

Commit message: Add files via upload

File: humanoid_arm_5dof/urdf/humanoid_arm_5dof.urdf (robot description, URDF)
Before this commit: robot humanoid_arm_5dof, 34 links, 33 joints
Links:
- link 1220_m4x16_left_shoulder_yaw_screws: mass 0.00141036418698186 -> 0.00141036418698184
- link left_elbow: mass 0.779765455773645 -> 0.779765456040378
- link left_elbow_rs03_actuator: mass 0.356550890896857 -> 0.35655089089686
- link left_elbow_rs03_flange: mass 0.0040755509739889 -> 0.00407555097398919
- link left_hand: mass 0.285530357235036 -> 0.285530357232192
- link left_hand_rs02: mass 0.180583065420555 -> 0.180583065420556
- link left_hand_rs02_flange: mass 0.00245793392108132 -> 0.00245793392108123
- link left_shoulder_pitch: mass 1.19772100042922 -> 1.19772099939528
- link left_shoulder_pitch_rs04_actuator: mass 0.517423577893352 -> 0.517423577893353
- link left_shoulder_pitch_rs04_flange: mass 0.00758352122244509 -> 0.00758352122244511
- link left_shoulder_roll: mass 0.997620687521854 -> 0.997620681307434
- link left_shoulder_roll_rs04_flange: mass 0.0075835212224449 -> 0.00758352122244512
- link left_shoulder_yaw: mass 0.488068654986572 -> 0.488068654987172
- link left_shoulder_yaw_flange: mass 0.0353531461099525 -> 0.035353146109953
- link left_shoulder_yaw_rs03_actuator: mass 0.3565509695881 -> 0.356550969588106
- link left_shoulder_yaw_rs03_flange: mass 0.00407555097398895 -> 0.00407555097398896
- link left_shoulder_yaw_shaft: mass 0.000903649674373941 -> 0.00090364967437399
- link left_wrist: mass 0.388950905166554 -> 0.388950905166551
- link left_wrist_actuator: mass 0.180583065420557 -> 0.180583065420556
- link left_wrist_rs02_flange: mass 0.0024579339210813 -> 0.00245793392108141
- link left_wrist_shaft: mass 0.000903649674373958 -> 0.000903649674373956
- link m3x16_left_hand_screws: mass 0.00139374174732655 -> 0.00139374174732656
- link m3x20_left_wrist_screws: mass 0.00162137028637934 -> 0.00162137028637932
- link m4x16_eft_elbow_screws: mass 0.00270184358647755 -> 0.00270184358647762
- link m4x16_left_shoulder_yaw_screws: mass 0.00270184474693415 -> 0.00270184474693414
- link m4x20_left_wrist_screws: mass 0.00232797016313307 -> 0.00232797016313296
- link m4x25_left_shoulder_screws_roll: mass 0.00451430348886335 -> 0.00451430348886334
- link m4x25_left_shoulder_yaw_screws: mass 0.00270858202481968 -> 0.00270858202481966
- link m5x22_screws_left_shoulder_pitch: mass 0.00474644340626607 -> 0.00474644340626584
- link m5x22_screws_left_shoulder_roll: mass 0.00610257053905752 -> 0.00610257053905775
Joints:
- joint left_elbow_rs03_joint: axis 0.442871169532446 0.896585259301625 0 -> 0.442871169532447 0.896585259301625 0
- joint left_shoulder_pitch_rs04_actuator_fixture_link: origin xyz=0.3827 -0.091826 1.4471 rpy=-0.54743 0 0 -> xyz=0 0.382699999999936 1.45000000000145 rpy=-0.61079662163343 0 1.57079632679489

Commit message: Add files via upload

File: humanoid_arm_5dof/urdf/humanoid_arm_5dof.urdf (robot description, URDF)
Before this commit: robot humanoid_arm_5dof, 34 links, 33 joints
Links:
- removed link 1220_m4x16_left_shoulder_yaw_screws
- removed link base_fixture_link
- removed link left_elbow_shaft
- removed link left_shoulder_yaw_shaft
- removed link left_wrist_shaft
- removed link m3x16_left_hand_screws
- removed link m3x20_left_wrist_screws
- removed link m4x16_eft_elbow_screws
- removed link m4x16_left_shoulder_yaw_screws
- removed link m4x20_left_wrist_screws
- removed link m4x25_left_elbow_screws
- removed link m4x25_left_shoulder_screws_roll
- removed link m4x25_left_shoulder_yaw_screws
- removed link m5x22_screws_left_shoulder_pitch
- removed link m5x22_screws_left_shoulder_roll
- added link base_link, mass 77.718; collision mesh filename=package://humanoid_arm_5dof/meshes/base_link.STL; visual mesh filename=package://humanoid_arm_5dof/meshes/base_link.STL
- added link left_palm, mass 0.047634; collision mesh filename=package://humanoid_arm_5dof/meshes/left_palm.STL; visual mesh filename=package://humanoid_arm_5dof/meshes/left_palm.STL
- added link left_palm_left_finger, mass 0.02913; collision mesh filename=package://humanoid_arm_5dof/meshes/left_palm_left_finger.STL; visual mesh filename=package://humanoid_arm_5dof/meshes/left_palm_left_finger.STL
- added link left_palm_right_finger, mass 0.02913; collision mesh filename=package://humanoid_arm_5dof/meshes/left_palm_right_finger.S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; visual mesh filename=package://humanoid_arm_5dof/meshes/left_palm_right_finger.S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
- link left_elbow: mass 0.779765456040378 -> 0.1949
- link left_elbow_rs03_actuator: mass 0.35655089089686 -> 0.83
- link left_elbow_rs03_flange: mass 0.00407555097398919 -> 0.005
- link left_hand: mass 0.285530357232192 -> 0.07138
- link left_hand_rs02: mass 0.180583065420556 -> 0.38
- link left_hand_rs02_flange: mass 0.00245793392108123 -> 0.0025
- link left_shoulder_pitch: mass 1.19772099939528 -> 0.29944
- link left_shoulder_pitch_rs04_actuator: mass 0.517423577893353 -> 1.345
- link left_shoulder_pitch_rs04_flange: mass 0.00758352122244511 -> 0.0075
- link left_shoulder_roll: mass 0.997620681307434 -> 0.2494
- link left_shoulder_roll_rs04_actuator: mass 0.517423577893355 -> 1.345
- link left_shoulder_roll_rs04_flange: mass 0.00758352122244512 -> 0.0075
- link left_shoulder_yaw: mass 0.488068654987172 -> 0.122018
- link left_shoulder_yaw_flange: mass 0.035353146109953 -> 0.008838
- link left_shoulder_yaw_rs03_actuator: mass 0.356550969588106 -> 0.83
- link left_shoulder_yaw_rs03_flange: mass 0.00407555097398896 -> 0.005
- link left_wrist: mass 0.388950905166551 -> 0.09723
- link left_wrist_actuator: mass 0.180583065420556 -> 0.38
- link left_wrist_rs02_flange: mass 0.00245793392108141 -> 0.0025
Joints:
- removed joint 1220_m4x16_left_shoulder_yaw_screws_fixture_joint
- removed joint left_elbow_fixture_joint
- removed joint left_elbow_rs03_joint
- removed joint left_elbow_shaft_fixture_joint
- removed joint left_hand_fixture_joint
- removed joint left_hand_rs02_joint
- removed joint left_shoulde_roll_fixture_joint
- removed joint left_shoulder_pitch_fixture_joint
- removed joint left_shoulder_pitch_rs04_joint
- removed joint left_shoulder_roll_rs04_flange_joint
- removed joint left_shoulder_roll_rs04_joint
- removed joint left_shoulder_yaw_fixture_joint
- removed joint left_shoulder_yaw_flange_fixture_joint
- removed joint left_shoulder_yaw_rs03_joint
- removed joint left_shoulder_yaw_shaft_fixture_joint
- removed joint left_wrist_actuator_fixture_link
- removed joint left_wrist_fixture_joint
- removed joint left_wrist_rs02_joint
- removed joint left_wrist_shaft_fixture_joint
- removed joint m3x16_left_hand_screws_fixture_joint
- removed joint m3x20_left_wrist_screws_fixture_joint
- removed joint m4x16_eft_elbow_screws_fixture_joint
- removed joint m4x16_left_shoulder_yaw_screws_fixture_joint
- removed joint m4x20_left_wrist_screws_fixture_joint
- removed joint m4x25_left_elbow_screws_fixture_joint
- removed joint m4x25_left_shoulder_screws_roll_fixture_joint
- removed joint m4x25_left_shoulder_yaw_screws_fixture_joint
- removed joint m5x22_screws_left_shoulder_pitch_fixture_joint
- removed joint m5x22_screws_left_shoulder_roll_fixture_joint
- added joint left_elbow_fixture: type fixed, parent left_elbow_rs03_flange, child left_elbow, origin xyz=0 0 0 rpy=0 0 0, axis 0 0 0
- added joint left_elbow_rs03: type revolute, parent left_elbow_rs03_actuator, child left_elbow_rs03_flange, origin xyz=0 0 0 rpy=0 0 0, axis -1 0 0, limit lower=-1.3 upper=1.9 effort=60 velocity=1.6
- added joint left_hand_fixture: type fixed, parent left_hand_rs02_flange, child left_hand, origin xyz=0 0 0 rpy=0 0 0, axis 0 0 0
- added joint left_hand_rs02: type revolute, parent left_hand_rs02, child left_hand_rs02_flange, origin xyz=0 0 0 rpy=0 0 0, axis 1 0 0, limit lower=-1.5 upper=1.7 effort=17 velocity=0.8
- added joint left_palm_fixture: type fixed, parent left_hand, child left_palm, origin xyz=0 0.046829 -0.045845 rpy=-0.77494 -0.017568 0.017203, axis 0 0 0
- added joint left_palm_left_finger: type prismatic, parent left_palm, child left_palm_left_finger, origin xyz=0 0 0 rpy=0 0 0, axis -1 0 0, limit lower=-0.0041 upper=0.033 effort=0 velocity=0
- added joint left_palm_right_finger: type prismatic, parent left_palm, child left_palm_right_finger, origin xyz=0 0 0 rpy=0 0 0, axis -1 0 0, limit lower=-0.033 upper=0.00026 effort=0 velocity=0
- added joint left_shoulde_roll_fixture: type fixed, parent left_shoulder_roll_rs04_actuator, child left_shoulder_roll, origin xyz=0 0 0 rpy=0 0 0, axis 0 0 0
- added joint left_shoulder_pitch_fixture: type fixed, parent left_shoulder_pitch_rs04_flange, child left_shoulder_pitch, origin xyz=0 0 0 rpy=0 0 0, axis 0 0 0
- added joint left_shoulder_pitch_rs04: type revolute, parent left_shoulder_pitch_rs04_actuator, child left_shoulder_pitch_rs04_flange, origin xyz=0 0 0 rpy=0 0 0, axis 1 0 0, limit lower=-3.14 upper=3.14 effort=120 velocity=3
- added joint left_shoulder_roll_rs04: type revolute, parent left_shoulder_roll_rs04_flange, child left_shoulder_roll_rs04_actuator, origin xyz=0 0 0 rpy=0 0 0, axis 0 -1 0, limit lower=-3.5 upper=0.6 effort=120 velocity=3
- added joint left_shoulder_roll_rs04_flange: type fixed, parent left_shoulder_pitch, child left_shoulder_roll_rs04_flange, origin xyz=0.11678 0.0487 -2.7056E-05 rpy=0 0 3.1416, axis 0 0 0
- added joint left_shoulder_yaw_fixture: type fixed, parent left_shoulder_yaw_flange, child left_shoulder_yaw, origin xyz=0 0 0 rpy=0 0 0, axis 0 0 0
- added joint left_shoulder_yaw_flange_fixture: type fixed, parent left_shoulder_yaw_rs03_flange, child left_shoulder_yaw_flange, origin xyz=0 0 0 rpy=0 0 0, axis 0 0 0
- added joint left_shoulder_yaw_rs03: type revolute, parent left_shoulder_yaw_rs03_actuator, child left_shoulder_yaw_rs03_flange, origin xyz=0 0 0 rpy=0 0 0, axis 0 0 1, limit lower=-3.14 upper=3.14 effort=60 velocity=1.6
- added joint left_wrist_fixture: type fixed, parent left_wrist_rs02_flange, child left_wrist, origin xyz=0 0 0 rpy=0 0 0, axis 0 0 0
- added joint left_wrist_rs02: type revolute, parent left_wrist_actuator, child left_wrist_rs02_flange, origin xyz=0 0 0 rpy=0 0 0, axis 0 1 0, limit lower=-3.14 upper=3.14 effort=17 velocity=0.8
- added joint left_wrist_rs02_actuator_fixture_link: type fixed, parent left_elbow, child left_wrist_actuator, origin xyz=0.0055 0.044061 -0.15849 rpy=-1.2996 0 0, axis 0 0 0
- joint left_elbow_rs03_actuator_ficture_link: origin xyz=0 0 0 rpy=0 0 0 -> xyz=0 0 -0.0987 rpy=0 0 0; parent m4x16_eft_elbow_screws -> left_shoulder_yaw
- joint left_hand_rs02_fixture_link: origin xyz=0 0 0 rpy=0 0 0 -> xyz=0 0.0945 0 rpy=0.64485 0.44406 0; parent m3x16_left_hand_screws -> left_wrist
- joint left_shoulder_pitch_rs04_actuator_fixture_link: origin xyz=0 0.382699999999936 1.45000000000145 rpy=-0.61079662163343 0 1.57079632679489 -> xyz=-0.1079 0 1.425 rpy=-0.67594 0 3.1416; parent base_fixture_link -> base_link
- joint left_shoulder_yaw_rs03_actuator_fixture_link: origin xyz=0 0 0 rpy=0 0 0 -> xyz=-0.021972 0.0377 -0.17358 rpy=0.057123 0.11257 0.47088; parent m4x16_left_shoulder_yaw_screws -> left_shoulder_roll
