Commit message: Add files via upload

File: humanoid_arm_5dof/urdf/humanoid_arm_5dof.urdf (robot description, URDF)
Before this commit: robot humanoid_arm_5dof, 23 links, 22 joints
Links:
- removed link left_hand_rs02
- removed link left_wrist_actuator
- added link left_hand_rs02_actuator, mass 0.38; collision mesh filename=package://humanoid_arm_5dof/meshes/left_hand_rs02_actuator.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; visual mesh filename=package://humanoid_arm_5dof/meshes/left_hand_rs02_actuator.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
- added link left_wrist_rs02_actuator, mass 0.38; collision mesh filename=package://humanoid_arm_5dof/meshes/left_wrist_rs02_actuator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; visual mesh filename=package://humanoid_arm_5dof/meshes/left_wrist_rs02_actuator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
- link left_elbow: mass 0.1949 -> 0.194942
- link left_palm_left_finger: mass 0.02913 -> 0.029134
- link left_palm_right_finger: mass 0.02913 -> 0.029134
- link left_shoulder_pitch: mass 0.29944 -> 0.298
- link left_shoulder_yaw: mass 0.122018 -> 0.12218
- link left_shoulder_yaw_rs03_actuator: mass 0.83 -> 830
- link left_wrist: mass 0.09723 -> 0.097238
Joints:
- removed joint left_elbow_rs03
- removed joint left_elbow_rs03_actuator_ficture_link
- removed joint left_hand_rs02
- removed joint left_hand_rs02_fixture_link
- removed joint left_shoulder_pitch_rs04
- removed joint left_shoulder_roll_rs04
- removed joint left_shoulder_yaw_rs03
- removed joint left_wrist_rs02
- added joint left_elbow_rs03_actuator_fixture_link: type fixed, parent left_shoulder_yaw, child left_elbow_rs03_actuator, origin xyz=0 0 -0.0987000004167597 rpy=0 0 0, axis 0 0 0
- added joint left_elbow_rs03_flange: type revolute, parent left_elbow_rs03_actuator, child left_elbow_rs03_flange, origin xyz=0 0 0 rpy=0 0 0, axis -1 0 0, limit lower=-1.3 upper=1.9 effort=60 velocity=1.6
- added joint left_hand_rs02_actuator_fixture_link: type fixed, parent left_wrist, child left_hand_rs02_actuator, origin xyz=0 0.0945 0 rpy=0.64485 0.44406 0, axis 0 0 0
- added joint left_hand_rs02_flange: type revolute, parent left_hand_rs02_actuator, child left_hand_rs02_flange, origin xyz=0 0 0 rpy=0 0 0, axis 0.999999999999735 0 0, limit lower=-1.5 upper=1.7 effort=17 velocity=0.8
- added joint left_shoulder_pitch_rs04_flange: type revolute, parent left_shoulder_pitch_rs04_actuator, child left_shoulder_pitch_rs04_flange, origin xyz=0 0 0 rpy=0 0 0, axis 1 0 0, limit lower=-3.14 upper=3.14 effort=120 velocity=3
- added joint left_shoulder_roll_rs04_actuator_fixture_link: type revolute, parent left_shoulder_roll_rs04_flange, child left_shoulder_roll_rs04_actuator, origin xyz=0 0 0 rpy=0 0 0, axis 0 -1 0, limit lower=-3.5 upper=0.6 effort=120 velocity=3
- added joint left_shoulder_yaw_rs03_flange: type revolute, parent left_shoulder_yaw_rs03_actuator, child left_shoulder_yaw_rs03_flange, origin xyz=0 0 0 rpy=0 0 0, axis 0 0 1, limit lower=-3.14 upper=3.14 effort=60 velocity=1.6
- added joint left_wrist_rs02_flange: type revolute, parent left_wrist_rs02_actuator, child left_wrist_rs02_flange, origin xyz=0 0 0 rpy=0 0 0, axis 0 1 0, limit lower=-3.14 upper=3.14 effort=17 velocity=0.8
- joint left_palm_fixture: origin xyz=0 0.046829 -0.045845 rpy=-0.77494 -0.017568 0.017203 -> xyz=0 0.0468292785877469 -0.0458451123506719 rpy=-0.774935929627841 -0.017568105500413 0.017202724160053
- joint left_shoulder_roll_rs04_flange: origin xyz=0.11678 0.0487 -2.7056E-05 rpy=0 0 3.1416 -> xyz=0.116775431275821 0.0487000000004332 -2.70558071411298E-05 rpy=0 0 3.14159265358979
- joint left_shoulder_yaw_rs03_actuator_fixture_link: origin xyz=-0.021972 0.0377 -0.17358 rpy=0.057123 0.11257 0.47088 -> xyz=-0.0219716026665047 0.037700000000231 -0.173578614834026 rpy=0.0571232415871479 0.112571267005327 0.470875575147914
- joint left_wrist_rs02_actuator_fixture_link: child left_wrist_actuator -> left_wrist_rs02_actuator

Commit message: Add files via upload

File: humanoid_arm_5dof/urdf/humanoid_arm_5dof.urdf (robot description, URDF)
Before this commit: robot humanoid_arm_5dof, 23 links, 22 joints
Links:
- link left_elbow: mass 0.194942 -> 0.1948
- link left_palm: mass 0.047634 -> 0.0476
- link left_palm_left_finger: mass 0.029134 -> 0.02912
- link left_palm_right_finger: mass 0.029134 -> 0.02912
- link left_shoulder_pitch: mass 0.298 -> 0.2994
- link left_shoulder_yaw: mass 0.12218 -> 0.122
- link left_shoulder_yaw_flange: mass 0.008838 -> 0.0088
- link left_shoulder_yaw_rs03_actuator: mass 830 -> 0.83
- link left_wrist: mass 0.097238 -> 0.09722
Joints:
- removed joint left_elbow_rs03_flange
- removed joint left_hand_rs02_flange
- removed joint left_shoulder_pitch_rs04_flange
- removed joint left_shoulder_roll_rs04_flange
- removed joint left_shoulder_yaw_rs03_flange
- removed joint left_wrist_rs02_flange
- added joint left_elbow_rs03: type revolute, parent left_elbow_rs03_actuator, child left_elbow_rs03_flange, origin xyz=0 0 0 rpy=0 0 0, axis -1 0 0, limit lower=-1.3 upper=1.9 effort=60 velocity=1.6
- added joint left_hand_rs02: type revolute, parent left_hand_rs02_actuator, child left_hand_rs02_flange, origin xyz=0 0 0 rpy=0 0 0, axis 0.999999999999735 0 0, limit lower=-1.5 upper=1.7 effort=17 velocity=0.8
- added joint left_shoulder_pitch_rs04: type revolute, parent left_shoulder_pitch_rs04_actuator, child left_shoulder_pitch_rs04_flange, origin xyz=0 0 0 rpy=0 0 0, axis 1 0 0, limit lower=-3.14 upper=3.14 effort=120 velocity=3
- added joint left_shoulder_roll_rs04: type fixed, parent left_shoulder_pitch, child left_shoulder_roll_rs04_flange, origin xyz=0.11678 0.0487 -2.7056E-05 rpy=0 0 3.1416, axis 0 0 0
- added joint left_shoulder_yaw_rs03: type revolute, parent left_shoulder_yaw_rs03_actuator, child left_shoulder_yaw_rs03_flange, origin xyz=0 0 0 rpy=0 0 0, axis 0 0 1, limit lower=-3.14 upper=3.14 effort=60 velocity=1.6
- added joint left_wrist_rs02: type revolute, parent left_wrist_rs02_actuator, child left_wrist_rs02_flange, origin xyz=0 0 0 rpy=0 0 0, axis 0 1 0, limit lower=-3.14 upper=3.14 effort=17 velocity=0.8
- joint left_hand_rs02_actuator_fixture_link: origin xyz=0 0.0945 0 rpy=0.64485 0.44406 0 -> xyz=0 0.0944999999997473 0 rpy=0.644846111175764 0.444064007774013 0
- joint left_wrist_rs02_actuator_fixture_link: origin xyz=0.0055 0.044061 -0.15849 rpy=-1.2996 0 0 -> xyz=0.00550000028936815 0.0440612514790653 -0.158489293351936 rpy=-1.29963429793404 0 0
